File: 0104-USB-HUB.kicad_sch (KiCad schematic)
At the start: 38 parts, among them J1 USB_US, J2 USB_DS, J3 USB_DS, J4 USB_DS, SW1 SW_Push_DPDT, SW2 SW_Push_DPDT, SW3 SW_Push_DPDT, U1 SL2.1A, Y1 12MHz

Commit message: Finish BOM
Parts:
- D4, D5, D6: Manufacturer (none) -> EVERLIGHT; PartNumber (none) -> C72041
- F1, F2, F3: value 2A/100ms -> 1.5A/3A; Manufacturer TLC -> BHFUSE; PartNumber C261954 -> C883133
- R1, R2: Manufacturer (none) -> UNI-ROYAL; PartNumber (none) -> C25905
- R3, R4, R5: Manufacturer (none) -> UNI-ROYAL; PartNumber (none) -> C4109
- U1: Manufacturer (none) -> CoreChips; PartNumber (none) -> C192893; Supplier JLC -> JLC-EXT
Changed lines of the file:
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@@
       (effects (font (size 1.27 1.27)) hide)
     )
-    (property "Manufacturer" "~" (id 4) (at 69.85 48.26 0)
-      (effects (font (size 1.27 1.27)) hide)
-    )
-    (property "PartNumber" "~" (id 5) (at 69.85 48.26 0)
+    (property "Manufacturer" "UNI-ROYAL" (id 4) (at 69.85 48.26 0)
+      (effects (font (size 1.27 1.27)) hide)
+    )
+    (property "PartNumber" "C25905" (id 5) (at 69.85 48.26 0)
       (effects (font (size 1.27 1.27)) hide)
     )
@@
       (effects (font (size 1.27 1.27)) hide)
     )
-    (property "Manufacturer" "~" (id 4) (at 224.79 114.3 0)
-      (effects (font (size 1.27 1.27)) hide)
-    )
-    (property "PartNumber" "~" (id 5) (at 224.79 114.3 0)
+    (property "Manufacturer" "UNI-ROYAL" (id 4) (at 224.79 114.3 0)
+      (effects (font (size 1.27 1.27)) hide)
+    )
+    (property "PartNumber" "C4109" (id 5) (at 224.79 114.3 0)
       (effects (font (size 1.27 1.27)) hide)
     )
@@
       (effects (font (size 1.27 1.27)) hide)
     )
-    (property "Manufacturer" "~" (id 4) (at 161.29 114.3 0)
-      (effects (font (size 1.27 1.27)) hide)
-    )
-    (property "PartNumber" "~" (id 5) (at 161.29 114.3 0)
+    (property "Manufacturer" "EVERLIGHT" (id 4) (at 161.29 114.3 0)
+      (effects (font (size 1.27 1.27)) hide)
+    )
+    (property "PartNumber" "C72041" (id 5) (at 161.29 114.3 0)
       (effects (font (size 1.27 1.27)) hide)
     )
@@
     (in_bom yes) (on_board yes) (fields_autoplaced)
     (property "Reference" "F1" (id 0) (at 62.23 107.95 90))
-    (property "Value" "2A/100ms" (id 1) (at 62.23 110.49 90))
+    (property "Value" "1.5A/3A" (id 1) (at 62.23 110.49 90))
     (property "Footprint" "Fuse:Fuse_1206_3216Metric" (id 2) (at 57.15 115.57 0)
       (effects (font (size 1.27 1.27)) (justify left) hide)
@@
       (effects (font (size 1.27 1.27)) hide)
     )
-    (property "Manufacturer" "TLC" (id 5) (at 62.23 114.3 0)
-      (effects (font (size 1.27 1.27)) hide)
-    )
-    (property "PartNumber" "C261954" (id 6) (at 62.23 114.3 0)
+    (property "Manufacturer" "BHFUSE" (id 5) (at 62.23 114.3 0)
+      (effects (font (size 1.27 1.27)) hide)
+    )
+    (property "PartNumber" "C883133" (id 6) (at 62.23 114.3 0)
       (effects (font (size 1.27 1.27)) hide)
     )
@@
       (effects (font (size 1.27 1.27)) hide)
     )
-    (property "Manufacturer" "~" (id 6) (at 85.09 114.3 0)
-      (effects (font (size 1.27 1.27)) hide)
-    )
-    (property "PartNumber" "~" (id 7) (at 85.09 114.3 0)
+    (property "Manufacturer" "EVERLIGHT" (id 6) (at 85.09 114.3 0)
+      (effects (font (size 1.27 1.27)) hide)
+    )
+    (property "PartNumber" "C72041" (id 7) (at 85.09 114.3 0)
       (effects (font (size 1.27 1.27)) hide)
     )
@@
       (effects (font (size 1.27 1.27)) hide)
     )
-    (property "Manufacturer" "~" (id 4) (at 238.76 53.34 0)
-      (effects (font (size 1.27 1.27)) hide)
-    )
-    (property "PartNumber" "~" (id 5) (at 238.76 53.34 0)
-      (effects (font (size 1.27 1.27)) hide)
-    )
-    (property "Supplier" "JLC" (id 6) (at 238.76 53.34 0)
+    (property "Manufacturer" "CoreChips" (id 4) (at 238.76 53.34 0)
+      (effects (font (size 1.27 1.27)) hide)
+    )
+    (property "PartNumber" "C192893" (id 5) (at 238.76 53.34 0)
+      (effects (font (size 1.27 1.27)) hide)
+    )
+    (property "Supplier" "JLC-EXT" (id 6) (at 238.76 53.34 0)
       (effects (font (size 1.27 1.27)) hide)
     )
@@
       (effects (font (size 1.27 1.27)) hide)
     )
-    (property "Manufacturer" "~" (id 6) (at 69.85 45.72 0)
-      (effects (font (size 1.27 1.27)) hide)
-    )
-    (property "PartNumber" "~" (id 7) (at 69.85 45.72 0)
+    (property "Manufacturer" "UNI-ROYAL" (id 6) (at 69.85 45.72 0)
+      (effects (font (size 1.27 1.27)) hide)
+    )
+    (property "PartNumber" "C25905" (id 7) (at 69.85 45.72 0)
       (effects (font (size 1.27 1.27)) hide)
     )
@@
       (effects (font (size 1.27 1.27)) hide)
     )
-    (property "Manufacturer" "~" (id 4) (at 237.49 114.3 0)
-      (effects (font (size 1.27 1.27)) hide)
-    )
-    (property "PartNumber" "~" (id 5) (at 237.49 114.3 0)
+    (property "Manufacturer" "EVERLIGHT" (id 4) (at 237.49 114.3 0)
+      (effects (font (size 1.27 1.27)) hide)
+    )
+    (property "PartNumber" "C72041" (id 5) (at 237.49 114.3 0)
       (effects (font (size 1.27 1.27)) hide)
     )
@@
       (effects (font (size 1.27 1.27)) hide)
     )
-    (property "Manufacturer" "~" (id 4) (at 148.59 114.3 0)
-      (effects (font (size 1.27 1.27)) hide)
-    )
-    (property "PartNumber" "~" (id 5) (at 148.59 114.3 0)
+    (property "Manufacturer" "UNI-ROYAL" (id 4) (at 148.59 114.3 0)
+      (effects (font (size 1.27 1.27)) hide)
+    )
+    (property "PartNumber" "C4109" (id 5) (at 148.59 114.3 0)
       (effects (font (size 1.27 1.27)) hide)
     )
@@
     (in_bom yes) (on_board yes) (fields_autoplaced)
     (property "Reference" "F3" (id 0) (at 214.63 107.95 90))
-    (property "Value" "2A/100ms" (id 1) (at 214.63 110.49 90))
+    (property "Value" "1.5A/3A" (id 1) (at 214.63 110.49 90))
     (property "Footprint" "Fuse:Fuse_1206_3216Metric" (id 2) (at 219.71 113.03 0)
       (effects (font (size 1.27 1.27)) (justify left) hide)
@@
       (effects (font (size 1.27 1.27)) hide)
     )
-    (property "Manufacturer" "TLC" (id 4) (at 214.63 114.3 0)
-      (effects (font (size 1.27 1.27)) hide)
-    )
-    (property "PartNumber" "C261954" (id 5) (at 214.63 114.3 0)
+    (property "Manufacturer" "BHFUSE" (id 4) (at 214.63 114.3 0)
+      (effects (font (size 1.27 1.27)) hide)
+    )
+    (property "PartNumber" "C883133" (id 5) (at 214.63 114.3 0)
       (effects (font (size 1.27 1.27)) hide)
     )
@@
     (in_bom yes) (on_board yes) (fields_autoplaced)
     (property "Reference" "F2" (id 0) (at 138.43 107.95 90))
-    (property "Value" "2A/100ms" (id 1) (at 138.43 110.49 90))
+    (property "Value" "1.5A/3A" (id 1) (at 138.43 110.49 90))
     (property "Footprint" "Fuse:Fuse_1206_3216Metric" (id 2) (at 143.51 113.03 0)
       (effects (font (size 1.27 1.27)) (justify left) hide)
@@
       (effects (font (size 1.27 1.27)) hide)
     )
-    (property "Manufacturer" "TLC" (id 4) (at 138.43 114.3 0)
-      (effects (font (size 1.27 1.27)) hide)
-    )
-    (property "PartNumber" "C261954" (id 5) (at 138.43 114.3 0)
+    (property "Manufacturer" "BHFUSE" (id 4) (at 138.43 114.3 0)
+      (effects (font (size 1.27 1.27)) hide)
+    )
+    (property "PartNumber" "C883133" (id 5) (at 138.43 114.3 0)
       (effects (font (size 1.27 1.27)) hide)
     )
@@
       (effects (font (size 1.27 1.27)) hide)
     )
-    (property "Manufacturer" "~" (id 6) (at 72.39 114.3 0)
-      (effects (font (size 1.27 1.27)) hide)
-    )
-    (property "PartNumber" "~" (id 7) (at 72.39 114.3 0)
+    (property "Manufacturer" "UNI-ROYAL" (id 6) (at 72.39 114.3 0)
+      (effects (font (size 1.27 1.27)) hide)
+    )
+    (property "PartNumber" "C4109" (id 7) (at 72.39 114.3 0)
       (effects (font (size 1.27 1.27)) hide)
     )
@@
     )
     (path "/885f053a-06c4-4626-b44e-950ada7246ee"
-      (reference "F1") (unit 1) (value "2A/100ms") (footprint "Fuse:Fuse_1206_3216Metric")
+      (reference "F1") (unit 1) (value "1.5A/3A") (footprint "Fuse:Fuse_1206_3216Metric")
     )
     (path "/f38e7857-1cb4-455a-bc26-8ac7e5eddd55"
-      (reference "F2") (unit 1) (value "2A/100ms") (footprint "Fuse:Fuse_1206_3216Metric")
+      (reference "F2") (unit 1) (value "1.5A/3A") (footprint "Fuse:Fuse_1206_3216Metric")
     )
     (path "/eb342539-2315-42c4-998f-702e9bdcf528"
-      (reference "F3") (unit 1) (value "2A/100ms") (footprint "Fuse:Fuse_1206_3216Metric")
+      (reference "F3") (unit 1) (value "1.5A/3A") (footprint "Fuse:Fuse_1206_3216Metric")
     )
     (path "/79e677ed-5dc9-43e0-9cef-8fad0f285323"

Commit message: Finish SCH
Connections:
- no-connect marks 14 -> 16
Other:
- company: (none) -> TileParts
- title: #0104 -> #0104 USB HUB
- moved on the sheet: D4, D5, D6, F1, F2, F3, R3, R4, R5, SW1, SW2, SW3
