File: 0104-USB-HUB.kicad_pcb (KiCad board)
At the start: 2 copper layers, 79.6 x 19.6 mm, 43 parts, among them J1 USB_US, J2 USB_DS, J3 USB_DS, J4 USB_DS, SW1 SW_Push_DPDT, SW2 SW_Push_DPDT, SW3 SW_Push_DPDT, U1 SL2.1A, Y1 12MHz

Commit message: Finish BOM
Parts:
- F1, F2, F3: value 2A/100ms -> 1.5A/3A
Changed lines of the file:
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@@
     (descr "LED SMD 0603 (1608 Metric), square (rectangular) end terminal, IPC_7351 nominal, (Body size source: http://www.tortai-tech.com/upload/download/2011102023233369053.pdf), generated with kicad-footprint-generator")
     (tags "LED")
-    (property "Manufacturer" "")
-    (property "PartNumber" "")
+    (property "Manufacturer" "EVERLIGHT")
+    (property "PartNumber" "C72041")
     (property "Sheetfile" "文件： 0104-USB-HUB.kicad_sch")
     (property "Sheetname" "")
@@
     (descr "Fuse SMD 1206 (3216 Metric), square (rectangular) end terminal, IPC_7351 nominal, (Body size source: http://www.tortai-tech.com/upload/download/2011102023233369053.pdf), generated with kicad-footprint-generator")
     (tags "fuse")
-    (property "Manufacturer" "TLC")
-    (property "PartNumber" "C261954")
+    (property "Manufacturer" "BHFUSE")
+    (property "PartNumber" "C883133")
     (property "Sheetfile" "文件： 0104-USB-HUB.kicad_sch")
     (property "Sheetname" "")
@@
       (effects (font (size 1 1) (thickness 0.15)))
     )
-    (fp_text value "2A/100ms" (at 0 1.82) (layer "F.Fab")
+    (fp_text value "1.5A/3A" (at 0 1.82) (layer "F.Fab")
       (effects (font (size 1 1) (thickness 0.15)))
     )
@@
     (descr "Resistor SMD 0402 (1005 Metric), square (rectangular) end terminal, IPC_7351 nominal, (Body size source: IPC-SM-782 page 72, https://www.pcb-3d.com/wordpress/wp-content/uploads/ipc-sm-782a_amendment_1_and_2.pdf), generated with kicad-footprint-generator")
     (tags "resistor")
-    (property "Manufacturer" "")
-    (property "PartNumber" "")
+    (property "Manufacturer" "UNI-ROYAL")
+    (property "PartNumber" "C4109")
     (property "Sheetfile" "文件： 0104-USB-HUB.kicad_sch")
     (property "Sheetname" "")
@@
     (descr "SOP, 16 Pin (https://www.diodes.com/assets/Datasheets/PAM8403.pdf), generated with kicad-footprint-generator ipc_gullwing_generator.py")
     (tags "SOP SO")
-    (property "Manufacturer" "")
-    (property "PartNumber" "")
-    (property "Sheetfile" "文件： 0104-USB-HUB.kicad_sch")
-    (property "Sheetname" "")
-    (property "Supplier" "JLC")
+    (property "Manufacturer" "CoreChips")
+    (property "PartNumber" "C192893")
+    (property "Sheetfile" "文件： 0104-USB-HUB.kicad_sch")
+    (property "Sheetname" "")
+    (property "Supplier" "JLC-EXT")
     (attr smd)
     (fp_text reference "U1" (at 0 -5.9) (layer "F.SilkS") hide
@@
     (descr "Resistor SMD 0402 (1005 Metric), square (rectangular) end terminal, IPC_7351 nominal, (Body size source: IPC-SM-782 page 72, https://www.pcb-3d.com/wordpress/wp-content/uploads/ipc-sm-782a_amendment_1_and_2.pdf), generated with kicad-footprint-generator")
     (tags "resistor")
-    (property "Manufacturer" "")
-    (property "PartNumber" "")
+    (property "Manufacturer" "UNI-ROYAL")
+    (property "PartNumber" "C4109")
     (property "Sheetfile" "文件： 0104-USB-HUB.kicad_sch")
     (property "Sheetname" "")
@@
     (descr "Resistor SMD 0402 (1005 Metric), square (rectangular) end terminal, IPC_7351 nominal, (Body size source: IPC-SM-782 page 72, https://www.pcb-3d.com/wordpress/wp-content/uploads/ipc-sm-782a_amendment_1_and_2.pdf), generated with kicad-footprint-generator")
     (tags "resistor")
-    (property "Manufacturer" "")
-    (property "PartNumber" "")
+    (property "Manufacturer" "UNI-ROYAL")
+    (property "PartNumber" "C4109")
     (property "Sheetfile" "文件： 0104-USB-HUB.kicad_sch")
     (property "Sheetname" "")
@@
     (descr "LED SMD 0603 (1608 Metric), square (rectangular) end terminal, IPC_7351 nominal, (Body size source: http://www.tortai-tech.com/upload/download/2011102023233369053.pdf), generated with kicad-footprint-generator")
     (tags "LED")
-    (property "Manufacturer" "")
-    (property "PartNumber" "")
+    (property "Manufacturer" "EVERLIGHT")
+    (property "PartNumber" "C72041")
     (property "Sheetfile" "文件： 0104-USB-HUB.kicad_sch")
     (property "Sheetname" "")
@@
     (descr "Fuse SMD 1206 (3216 Metric), square (rectangular) end terminal, IPC_7351 nominal, (Body size source: http://www.tortai-tech.com/upload/download/2011102023233369053.pdf), generated with kicad-footprint-generator")
     (tags "fuse")
-    (property "Manufacturer" "TLC")
-    (property "PartNumber" "C261954")
+    (property "Manufacturer" "BHFUSE")
+    (property "PartNumber" "C883133")
     (property "Sheetfile" "文件： 0104-USB-HUB.kicad_sch")
     (property "Sheetname" "")
@@
       (effects (font (size 1 1) (thickness 0.15)))
     )
-    (fp_text value "2A/100ms" (at 0 1.82) (layer "F.Fab")
+    (fp_text value "1.5A/3A" (at 0 1.82) (layer "F.Fab")
       (effects (font (size 1 1) (thickness 0.15)))
     )
@@
     (descr "Fuse SMD 1206 (3216 Metric), square (rectangular) end terminal, IPC_7351 nominal, (Body size source: http://www.tortai-tech.com/upload/download/2011102023233369053.pdf), generated with kicad-footprint-generator")
     (tags "fuse")
-    (property "Manufacturer" "TLC")
-    (property "PartNumber" "C261954")
+    (property "Manufacturer" "BHFUSE")
+    (property "PartNumber" "C883133")
     (property "Sheetfile" "文件： 0104-USB-HUB.kicad_sch")
     (property "Sheetname" "")
@@
       (effects (font (size 1 1) (thickness 0.15)))
     )
-    (fp_text value "2A/100ms" (at 0 1.82) (layer "F.Fab")
+    (fp_text value "1.5A/3A" (at 0 1.82) (layer "F.Fab")
       (effects (font (size 1 1) (thickness 0.15)))
     )
@@
     (descr "Resistor SMD 0402 (1005 Metric), square (rectangular) end terminal, IPC_7351 nominal, (Body size source: IPC-SM-782 page 72, https://www.pcb-3d.com/wordpress/wp-content/uploads/ipc-sm-782a_amendment_1_and_2.pdf), generated with kicad-footprint-generator")
     (tags "resistor")
-    (property "Manufacturer" "")
-    (property "PartNumber" "")
+    (property "Manufacturer" "UNI-ROYAL")
+    (property "PartNumber" "C25905")
     (property "Sheetfile" "文件： 0104-USB-HUB.kicad_sch")
     (property "Sheetname" "")
@@
     (descr "Resistor SMD 0402 (1005 Metric), square (rectangular) end terminal, IPC_7351 nominal, (Body size source: IPC-SM-782 page 72, https://www.pcb-3d.com/wordpress/wp-content/uploads/ipc-sm-782a_amendment_1_and_2.pdf), generated with kicad-footprint-generator")
     (tags "resistor")
-    (property "Manufacturer" "")
-    (property "PartNumber" "")
+    (property "Manufacturer" "UNI-ROYAL")
+    (property "PartNumber" "C25905")
     (property "Sheetfile" "文件： 0104-USB-HUB.kicad_sch")
     (property "Sheetname" "")
@@
     (descr "LED SMD 0603 (1608 Metric), square (rectangular) end terminal, IPC_7351 nominal, (Body size source: http://www.tortai-tech.com/upload/download/2011102023233369053.pdf), generated with kicad-footprint-generator")
     (tags "LED")
-    (property "Manufacturer" "")
-    (property "PartNumber" "")
-    (property "Sheetfile" "文件： 0104-USB-HUB.kicad_sch")
-    (property "Sheetname" "")
+    (property "Manufacturer" "EVERLIGHT")
+    (property "PartNumber" "C72041")
+    (property "Sheetfile" "文件： 0104-USB-HUB.kicad_sch")
+    (property "Sheetname" "")

Commit message: Output docs
Parts:
- added REF**: JLC_CRAFT_EDGE, JLC-SMT:JLC_CRAFT_EDGE_3P, F.Cu at (176.5, 100.2)
- added REF**: JLC_CRAFT_EDGE, JLC-SMT:JLC_CRAFT_EDGE_3P, F.Cu at (103.5, 100.2)
- added REF**: JLC_CRAFT_EDGE, JLC-SMT:JLC_CRAFT_EDGE_3P, F.Cu at (176.5, 119.8)
- added REF**: JLC_CRAFT_EDGE, JLC-SMT:JLC_CRAFT_EDGE_3P, F.Cu at (103.5, 119.8)
Routing:
- net GND: vias 169 -> 164
Other:
- board size 79.6 x 19.6 mm -> 79.6 x 35 mm
- board text added: "JLCJLCJLCJLC"
